File: Power.sch (KiCad schematic (older format))
At the start: 11 parts

Commit message: Current/Fan updates
Parts:
- removed F? (x4): FUSE, ~, symbol FUSE
- added TH? (x4): THERMISTOR, ~, symbol THERMISTOR
Connections:
- net +12P: now also TH?.2
- net +3.3V: now also TH?.2
- net +5V: now also TH?.2
- net -12P: now also TH?.2
- net +12C: now reaches P?.10 (P10)
- net +12C: now also TH?.1
- net at P?.14 (P14): now also TH?.1
- net at P?.2 (P2): now also TH?.1
- net at P?.4 (P4), P?.6 (P6): now also TH?.1
Changed lines of the file:
@@
 Sheet 4 9
 Title ""
-Date "12 feb 2014"
+Date "13 feb 2014"
 Rev ""
 Comp ""
@@
 $EndComp
 $Comp
-L FUSE F?
-U 1 1 52F7202A
-P 3500 1650
-F 0 "F?" H 3600 1700 40  0000 C CNN
-F 1 "FUSE" H 3400 1600 40  0000 C CNN
-F 2 "~" H 3500 1650 60  0000 C CNN
-F 3 "~" H 3500 1650 60  0000 C CNN
-	1    3500 1650
-	1    0    0    -1
-$EndComp
-$Comp
-L FUSE F?
-U 1 1 52F72037
-P 4300 1850
-F 0 "F?" H 4400 1900 40  0000 C CNN
-F 1 "FUSE" H 4200 1800 40  0000 C CNN
-F 2 "~" H 4300 1850 60  0000 C CNN
-F 3 "~" H 4300 1850 60  0000 C CNN
-	1    4300 1850
-	1    0    0    -1
-$EndComp
-$Comp
-L FUSE F?
-U 1 1 52F7203D
-P 4950 2050
-F 0 "F?" H 5050 2100 40  0000 C CNN
-F 1 "FUSE" H 4850 2000 40  0000 C CNN
-F 2 "~" H 4950 2050 60  0000 C CNN
-F 3 "~" H 4950 2050 60  0000 C CNN
-	1    4950 2050
-	1    0    0    -1
-$EndComp
-$Comp
-L FUSE F?
-U 1 1 52F72043
-P 5650 2250
-F 0 "F?" H 5750 2300 40  0000 C CNN
-F 1 "FUSE" H 5550 2200 40  0000 C CNN
-F 2 "~" H 5650 2250 60  0000 C CNN
-F 3 "~" H 5650 2250 60  0000 C CNN
-	1    5650 2250
-	1    0    0    -1
-$EndComp
-$Comp
 L SWITCH_INV SW?
 U 1 1 52F7204B
@@
 $EndComp
 Wire Wire Line
-	2950 1650 3250 1650
-Wire Wire Line
-	3750 1650 4250 1650
+	2950 1650 3450 1650
+Wire Wire Line
+	3950 1650 4250 1650
 Wire Wire Line
 	4250 1650 4250 1150
@@
 	6050 2250 5900 2250
 Wire Wire Line
-	2150 1750 1050 1750
+	1050 1750 2150 1750
 Wire Wire Line
 	2150 1850 1700 1850
@@
 	9300 3550 9300 3800
 Connection ~ 8450 3550
+Wire Wire Line
+	3300 1250 3300 2050
+Connection ~ 3300 2050
+$Comp
+L +12C #PWR?
+U 1 1 52FC4237
+P 3300 1250
+F 0 "#PWR?" H 3300 1220 30  0001 C CNN
+F 1 "+12C" H 3300 1360 40  0000 C CNN
+F 2 "" H 3300 1250 60  0000 C CNN
+F 3 "" H 3300 1250 60  0000 C CNN
+	1    3300 1250
+	1    0    0    -1
+$EndComp
+$Comp
+L THERMISTOR TH?
+U 1 1 52FC4C2B
+P 3700 1650
+F 0 "TH?" V 3800 1700 50  0000 C CNN
+F 1 "THERMISTOR" V 3600 1650 50  0000 C CNN
+F 2 "~" H 3700 1650 60  0000 C CNN
+F 3 "~" H 3700 1650 60  0000 C CNN
+	1    3700 1650
+	0    -1   -1   0
+$EndComp
+$Comp
+L THERMISTOR TH?
+U 1 1 52FC4C38
+P 4300 1850
+F 0 "TH?" V 4400 1900 50  0000 C CNN
+F 1 "THERMISTOR" V 4200 1850 50  0000 C CNN
+F 2 "~" H 4300 1850 60  0000 C CNN
+F 3 "~" H 4300 1850 60  0000 C CNN
+	1    4300 1850
+	0    -1   -1   0
+$EndComp
+$Comp
+L THERMISTOR TH?
+U 1 1 52FC4C3E
+P 4950 2050
+F 0 "TH?" V 5050 2100 50  0000 C CNN
+F 1 "THERMISTOR" V 4850 2050 50  0000 C CNN
+F 2 "~" H 4950 2050 60  0000 C CNN
+F 3 "~" H 4950 2050 60  0000 C CNN
+	1    4950 2050
+	0    -1   -1   0
+$EndComp
+$Comp
+L THERMISTOR TH?
+U 1 1 52FC4C44
+P 5650 2250
+F 0 "TH?" V 5750 2300 50  0000 C CNN
+F 1 "THERMISTOR" V 5550 2250 50  0000 C CNN
+F 2 "~" H 5650 2250 60  0000 C CNN
+F 3 "~" H 5650 2250 60  0000 C CNN
+	1    5650 2250
+	0    -1   -1   0
+$EndComp
 $EndSCHEMATC
